Commit message: initial2

File: ur10e_hande_description/urdf/ur10e_hande_description_macro.xacro (robot description, xacro)
@@ -2,6 +2,6 @@
 <robot xmlns:xacro="http://ros.org/wiki/xacro">
   <xacro:include filename="$(find ur_description)/urdf/ur_macro.xacro"/>
-  <xacro:include filename="$(find hande_description)/urdf/robotiq_hande_gripper.xacro"/>
-  <xacro:macro name="ur10e_hande" params="
+  <xacro:include filename="$(find hande_description)/urdf/robotiq_hande_gripper.xacro"/> <!-- 그리퍼 추가 -->
+  <xacro:macro name="ur10e_hande_robot" params="
     parent
     *origin
@@ -11,18 +11,21 @@
     physical_parameters_file
     visual_parameters_file
+    use_fake_hardware
     ">
-    <!-- UR10e 로봇 생성 -->
+    <!--This will create the specific robot-->
     <xacro:ur_robot
       name="${ur_type}"
       tf_prefix=""
-      parent="${parent}"
+      parent="world"
       joint_limits_parameters_file="${joint_limits_parameters_file}"
       kinematics_parameters_file="${kinematics_parameters_file}"
       physical_parameters_file="${physical_parameters_file}"
       visual_parameters_file="${visual_parameters_file}"
+      use_fake_hardware="false"
+      use_tool_communication="true"
+      generate_ros2_control_tag="true"
     >
-      <xacro:insert_block name="origin"/>
+      <origin xyz="0 0 0" rpy="0 0 0" />
     </xacro:ur_robot>
-    <!-- Hand-E 그리퍼를 tool0에 연결 (올바른 매크로 이름) -->
     <xacro:robotiq_hande_gripper
       name="robotiq_hande_gripper"
@@ -37,5 +40,5 @@
       stop_bit="1"
       slave_id="9"
-      use_fake_hardware="true"
+      use_fake_hardware="${use_fake_hardware}"
     />
   </xacro:macro>

File: ur10e_hande_moveit_config/config/ur10e_hande_robot.ros2_control.xacro (robot description, xacro)
@@ -1,5 +1,5 @@
 <?xml version="1.0"?>
 <robot xmlns:xacro="http://www.ros.org/wiki/xacro">
-    <xacro:macro name="ur10e_hande_ros2_control" params="name initial_positions_file">
+    <xacro:macro name="ur10e_hande_robot_ros2_control" params="name initial_positions_file">
         <xacro:property name="initial_positions" value="${load_yaml(initial_positions_file)['initial_positions']}"/>
         <ros2_control name="${name}" type="system">
@@ -8,11 +8,4 @@
                 <plugin>mock_components/GenericSystem</plugin>
             </hardware>
-            <joint name="robotiq_hande_left_finger_joint">
-                <command_interface name="position"/>
-                <state_interface name="position">
-                  <param name="initial_value">${initial_positions['robotiq_hande_left_finger_joint']}</param>
-                </state_interface>
-                <state_interface name="velocity"/>
-            </joint>
             <joint name="shoulder_pan_joint">
                 <command_interface name="position"/>
@@ -57,4 +50,11 @@
                 <state_interface name="velocity"/>
             </joint>
+            <joint name="robotiq_hande_left_finger_joint">
+                <command_interface name="position"/>
+                <state_interface name="position">
+                  <param name="initial_value">${initial_positions['robotiq_hande_left_finger_joint']}</param>
+                </state_interface>
+                <state_interface name="velocity"/>
+            </joint>
         </ros2_control>
     </xacro:macro>
