Commit message: initialized

File: ur10e_hande_description/urdf/ur10e_hande_description.urdf.xacro (robot description, xacro)
@@ -8,4 +8,6 @@
   <xacro:arg name="visual_parameters_file" default="$(find ur_description)/config/$(arg ur_type)/visual_parameters.yaml"/>
   <xacro:arg name="use_fake_hardware" default="true"/>
+  <xacro:arg name="ur_prefix" default="ur_"/>
+  <xacro:arg name="gripper_prefix" default="gr_"/>
   <link name="world"/>
   <!--This will create the scene where the robot is located in-->
@@ -18,4 +20,6 @@
     visual_parameters_file="$(arg visual_parameters_file)"
     use_fake_hardware="$(arg use_fake_hardware)"
+    ur_prefix="$(arg ur_prefix)"
+    gripper_prefix="$(arg gripper_prefix)"
     >
       <origin xyz="0 0 1" rpy="0 0 0" />

File: ur10e_hande_description/urdf/ur10e_hande_description_macro.xacro (robot description, xacro)
@@ -1,6 +1,7 @@
 <?xml version="1.0"?>
+<!-- macro.xacro 는 아주 기본적인 로봇 세팅 파일. urdf.xacro는 macro.xacro에서 세팅에 필요한 인자를 주고 스폰시키는 완성 파일. -->
 <robot xmlns:xacro="http://ros.org/wiki/xacro">
   <xacro:include filename="$(find ur_description)/urdf/ur_macro.xacro"/>
-  <xacro:include filename="$(find hande_description)/urdf/robotiq_hande_gripper.xacro"/> <!-- 그리퍼 추가 -->
+  <xacro:include filename="$(find hande_description)/urdf/hande_gripper.xacro"/> <!-- 그리퍼 추가 -->
   <xacro:macro name="ur10e_hande_robot" params="
     parent
@@ -12,9 +13,12 @@
     visual_parameters_file
     use_fake_hardware
+    ur_prefix
+    gripper_prefix
     ">
-    <!--This will create the specific robot-->
+    <!-- 네임스페이스 = MANIPULATOR, GRIPPER -->
+    <!-- fake_hardware 사용 가능              -->
     <xacro:ur_robot
       name="${ur_type}"
-      tf_prefix=""
+      tf_prefix="${ur_prefix}"
       parent="world"
       joint_limits_parameters_file="${joint_limits_parameters_file}"
@@ -28,8 +32,8 @@
       <origin xyz="0 0 0" rpy="0 0 0" />
     </xacro:ur_robot>
-    <xacro:robotiq_hande_gripper
-      name="robotiq_hande_gripper"
-      prefix=""
-      parent="tool0"
+    <xacro:hande_gripper
+      name="hande_gripper"
+      prefix="${gripper_prefix}"
+      parent="${ur_prefix}tool0"
       grip_pos_min="0"
       grip_pos_max="0.025"

File: ur10e_hande_moveit_config/config/ur10e_hande_robot.ros2_control.xacro (robot description, xacro)
@@ -1,57 +1,57 @@
 <?xml version="1.0"?>
-<robot xmlns:xacro="http://ros.org/wiki/xacro">
-    <xacro:macro name="ur10e_hande_robot_ros2_control" params="name initial_positions_file use_fake_hardware">
+<robot xmlns:xacro="http://www.ros.org/wiki/xacro">
+    <xacro:macro name="ur10e_hande_robot_ros2_control" params="name initial_positions_file">
         <xacro:property name="initial_positions" value="${load_yaml(initial_positions_file)['initial_positions']}"/>
         <ros2_control name="${name}" type="system">
             <hardware>
-                <xacro:if value="${use_fake_hardware}">
-                    <plugin>mock_components/GenericSystem</plugin>
-                </xacro:if>
-                <xacro:unless value="${use_fake_hardware}">
-                    <!-- 실제 하드웨어에서는 UR 드라이버가 UR 조인트를 관리 -->
-                    <!-- 그리퍼는 별도 드라이버에서 관리 -->
-                    <plugin>mock_components/GenericSystem</plugin>
-                </xacro:unless>
+                <!-- By default, set up controllers for simulation. This won't work on real hardware -->
+                <plugin>mock_components/GenericSystem</plugin>
             </hardware>
-            <!-- UR 조인트들 -->
-            <joint name="shoulder_pan_joint">
+            <joint name="ur_shoulder_pan_joint">
                 <command_interface name="position"/>
                 <state_interface name="position">
-                  <param name="initial_value">${initial_positions['shoulder_pan_joint']}</param>
+                  <param name="initial_value">${initial_positions['ur_shoulder_pan_joint']}</param>
                 </state_interface>
                 <state_interface name="velocity"/>
             </joint>
-            <joint name="shoulder_lift_joint">
+            <joint name="ur_shoulder_lift_joint">
                 <command_interface name="position"/>
                 <state_interface name="position">
-                  <param name="initial_value">${initial_positions['shoulder_lift_joint']}</param>
+                  <param name="initial_value">${initial_positions['ur_shoulder_lift_joint']}</param>
                 </state_interface>
                 <state_interface name="velocity"/>
             </joint>
-            <joint name="elbow_joint">
+            <joint name="ur_elbow_joint">
                 <command_interface name="position"/>
                 <state_interface name="position">
-                  <param name="initial_value">${initial_positions['elbow_joint']}</param>
+                  <param name="initial_value">${initial_positions['ur_elbow_joint']}</param>
                 </state_interface>
                 <state_interface name="velocity"/>
             </joint>
-            <joint name="wrist_1_joint">
+            <joint name="ur_wrist_1_joint">
                 <command_interface name="position"/>
                 <state_interface name="position">
-                  <param name="initial_value">${initial_positions['wrist_1_joint']}</param>
+                  <param name="initial_value">${initial_positions['ur_wrist_1_joint']}</param>
                 </state_interface>
                 <state_interface name="velocity"/>
             </joint>
-            <joint name="wrist_2_joint">
+            <joint name="ur_wrist_2_joint">
                 <command_interface name="position"/>
                 <state_interface name="position">
-                  <param name="initial_value">${initial_positions['wrist_2_joint']}</param>
+                  <param name="initial_value">${initial_positions['ur_wrist_2_joint']}</param>
                 </state_interface>
                 <state_interface name="velocity"/>
             </joint>
-            <joint name="wrist_3_joint">
+            <joint name="ur_wrist_3_joint">
                 <command_interface name="position"/>
                 <state_interface name="position">
-                  <param name="initial_value">${initial_positions['wrist_3_joint']}</param>
+                  <param name="initial_value">${initial_positions['ur_wrist_3_joint']}</param>
+                </state_interface>
+                <state_interface name="velocity"/>
+            </joint>
+            <joint name="gr_hande_left_finger_joint">
+                <command_interface name="position"/>
+                <state_interface name="position">
+                  <param name="initial_value">${initial_positions['gr_hande_left_finger_joint']}</param>
                 </state_interface>
                 <state_interface name="velocity"/>

File: ur10e_hande_moveit_config/config/ur10e_hande_robot.urdf.xacro (robot description, xacro)
@@ -1,13 +1,9 @@
 <?xml version="1.0"?>
-<robot xmlns:xacro="http://ros.org/wiki/xacro" name="ur10e_hande_robot">
+<robot xmlns:xacro="http://www.ros.org/wiki/xacro" name="ur10e_hande_robot">
     <xacro:arg name="initial_positions_file" default="initial_positions.yaml" />
-    <xacro:arg name="use_fake_hardware" default="true" />
     <!-- Import ur10e_hande_robot urdf file -->
     <xacro:include filename="$(find ur10e_hande_description)/urdf/ur10e_hande_description.urdf.xacro" />
     <!-- Import control_xacro -->
     <xacro:include filename="ur10e_hande_robot.ros2_control.xacro" />
-    <xacro:ur10e_hande_robot_ros2_control
-        name="FakeSystem"
-        initial_positions_file="$(arg initial_positions_file)"
-        use_fake_hardware="$(arg use_fake_hardware)"/>
+    <xacro:ur10e_hande_robot_ros2_control name="FakeSystem" initial_positions_file="$(arg initial_positions_file)"/>
 </robot>
