Commit message: build ur10e-hande

File: ur10e_hande_moveit_config/config/ur10e_hande_robot.ros2_control.xacro (robot description, xacro)
@@ -1,11 +1,18 @@
 <?xml version="1.0"?>
-<robot xmlns:xacro="http://www.ros.org/wiki/xacro">
-    <xacro:macro name="ur10e_hande_robot_ros2_control" params="name initial_positions_file">
+<robot xmlns:xacro="http://ros.org/wiki/xacro">
+    <xacro:macro name="ur10e_hande_robot_ros2_control" params="name initial_positions_file use_fake_hardware">
         <xacro:property name="initial_positions" value="${load_yaml(initial_positions_file)['initial_positions']}"/>
         <ros2_control name="${name}" type="system">
             <hardware>
-                <!-- By default, set up controllers for simulation. This won't work on real hardware -->
-                <plugin>mock_components/GenericSystem</plugin>
+                <xacro:if value="${use_fake_hardware}">
+                    <plugin>mock_components/GenericSystem</plugin>
+                </xacro:if>
+                <xacro:unless value="${use_fake_hardware}">
+                    <!-- 실제 하드웨어에서는 UR 드라이버가 UR 조인트를 관리 -->
+                    <!-- 그리퍼는 별도 드라이버에서 관리 -->
+                    <plugin>mock_components/GenericSystem</plugin>
+                </xacro:unless>
             </hardware>
+            <!-- UR 조인트들 -->
             <joint name="shoulder_pan_joint">
                 <command_interface name="position"/>
@@ -50,4 +57,5 @@
                 <state_interface name="velocity"/>
             </joint>
+            <!-- Hande 그리퍼 조인트 (2F-140 드라이버와 호환) -->
             <joint name="robotiq_hande_left_finger_joint">
                 <command_interface name="position"/>

File: ur10e_hande_moveit_config/config/ur10e_hande_robot.urdf.xacro (robot description, xacro)
@@ -1,9 +1,13 @@
 <?xml version="1.0"?>
-<robot xmlns:xacro="http://www.ros.org/wiki/xacro" name="ur10e_hande_robot">
+<robot xmlns:xacro="http://ros.org/wiki/xacro" name="ur10e_hande_robot">
     <xacro:arg name="initial_positions_file" default="initial_positions.yaml" />
+    <xacro:arg name="use_fake_hardware" default="true" />
     <!-- Import ur10e_hande_robot urdf file -->
     <xacro:include filename="$(find ur10e_hande_description)/urdf/ur10e_hande_description.urdf.xacro" />
     <!-- Import control_xacro -->
     <xacro:include filename="ur10e_hande_robot.ros2_control.xacro" />
-    <xacro:ur10e_hande_robot_ros2_control name="FakeSystem" initial_positions_file="$(arg initial_positions_file)"/>
+    <xacro:ur10e_hande_robot_ros2_control
+        name="FakeSystem"
+        initial_positions_file="$(arg initial_positions_file)"
+        use_fake_hardware="$(arg use_fake_hardware)"/>
 </robot>
