Commit message: test

File: hande_description/urdf/robotiq_hande_gripper.xacro (robot description, xacro)
@@ -106,5 +106,5 @@
       <axis xyz="-1 0 0"/>
       <limit effort="130" lower="${grip_pos_min}" upper="${grip_pos_max}" velocity="0.15"/>
-      <!-- <mimic joint="${prefix}robotiq_hande_left_finger_joint" multiplier="1" offset="0"/> -->
+      <mimic joint="${prefix}robotiq_hande_left_finger_joint" />
     </joint>
     <link name="${prefix}robotiq_hande_right_finger">

File: ur10e_hande_moveit_config/config/ur10e_hande_robot.ros2_control.xacro (robot description, xacro)
@@ -57,19 +57,4 @@
                 <state_interface name="velocity"/>
             </joint>
-            <!-- Hande 그리퍼 조인트 (2F-140 드라이버와 호환) -->
-            <joint name="robotiq_hande_left_finger_joint">
-                <command_interface name="position"/>
-                <state_interface name="position">
-                  <param name="initial_value">${initial_positions['robotiq_hande_left_finger_joint']}</param>
-                </state_interface>
-                <state_interface name="velocity"/>
-            </joint>
-            <joint name="robotiq_hande_right_finger_joint">
-                <command_interface name="position"/>
-                <state_interface name="position">
-                  <param name="initial_value">${initial_positions['robotiq_hande_left_finger_joint']}</param>
-                </state_interface>
-                <state_interface name="velocity"/>
-            </joint>
         </ros2_control>
     </xacro:macro>
