Commit message: NEWNEW

File: hande_description/urdf/hande_gripper.ros2_control.xacro (robot description, xacro)
@@ -32,4 +32,16 @@
         </state_interface>
       </joint>
+      <joint name="${prefix}hande_right_finger_joint">
+        <command_interface name="position">
+          <param name="min">0</param>
+          <param name="max">0.025</param>
+        </command_interface>
+        <state_interface name="position">
+          <param name="initial_value">0.025</param>
+        </state_interface>
+        <state_interface name="velocity">
+          <param name="initial_value">0</param>
+        </state_interface>
+      </joint>
     </ros2_control>
   </xacro:macro>

File: hande_description/urdf/hande_gripper.xacro (robot description, xacro)
@@ -5,19 +5,5 @@
   -->
   <xacro:include filename="$(find hande_description)/urdf/hande_gripper.ros2_control.xacro"/>
-  <!-- Cylinder inertial macro integrated -->
-  <xacro:macro name="__hande_cylinder_inertial" params="radius height mass *origin">
-    <inertial>
-      <mass value="${mass}"/>
-      <xacro:insert_block name="origin"/>
-      <inertia
-        ixx="${0.0833333 * mass * (3 * (radius * radius) + height * height)}"
-        ixy="0.0"
-        ixz="0.0"
-        iyy="${0.0833333 * mass * (3 * (radius * radius) + height * height)}"
-        iyz="0.0"
-        izz="${0.5 * mass * (radius * radius)}"
-      />
-    </inertial>
-  </xacro:macro>
+  <xacro:include filename="$(find hande_description)/urdf/cylinder_inertial.xacro"/>
   <xacro:macro name="hande_gripper" params="name prefix parent grip_pos_min grip_pos_max tty baudrate parity data_bits stop_bit slave_id use_fake_hardware coupler_mass:=0.119">
     <!-- ros2_control parameters  -->
@@ -120,5 +106,5 @@
       <axis xyz="-1 0 0"/>
       <limit effort="130" lower="${grip_pos_min}" upper="${grip_pos_max}" velocity="0.15"/>
-      <mimic joint="${prefix}hande_left_finger_joint" multiplier="1" offset="0"/>
+      <!-- <mimic joint="${prefix}hande_left_finger_joint" multiplier="1" offset="0"/> -->
     </joint>
     <link name="${prefix}hande_right_finger">

File: ur10e_hande_description/urdf/ur10e_hande_description.urdf.xacro (robot description, xacro)
@@ -8,6 +8,4 @@
   <xacro:arg name="visual_parameters_file" default="$(find ur_description)/config/$(arg ur_type)/visual_parameters.yaml"/>
   <xacro:arg name="use_fake_hardware" default="true"/>
-  <xacro:arg name="ur_prefix" default="ur_"/>
-  <xacro:arg name="gripper_prefix" default="gr_"/>
   <link name="world"/>
   <!--This will create the scene where the robot is located in-->
@@ -20,6 +18,4 @@
     visual_parameters_file="$(arg visual_parameters_file)"
     use_fake_hardware="$(arg use_fake_hardware)"
-    ur_prefix="$(arg ur_prefix)"
-    gripper_prefix="$(arg gripper_prefix)"
     >
       <origin xyz="0 0 1" rpy="0 0 0" />

File: ur10e_hande_description/urdf/ur10e_hande_description_macro.xacro (robot description, xacro)
@@ -1,4 +1,3 @@
 <?xml version="1.0"?>
-<!-- macro.xacro 는 아주 기본적인 로봇 세팅 파일. urdf.xacro는 macro.xacro에서 세팅에 필요한 인자를 주고 스폰시키는 완성 파일. -->
 <robot xmlns:xacro="http://ros.org/wiki/xacro">
   <xacro:include filename="$(find ur_description)/urdf/ur_macro.xacro"/>
@@ -13,12 +12,9 @@
     visual_parameters_file
     use_fake_hardware
-    ur_prefix
-    gripper_prefix
     ">
-    <!-- 네임스페이스 = MANIPULATOR, GRIPPER -->
-    <!-- fake_hardware 사용 가능              -->
+    <!--This will create the specific robot-->
     <xacro:ur_robot
       name="${ur_type}"
-      tf_prefix="${ur_prefix}"
+      tf_prefix=""
       parent="world"
       joint_limits_parameters_file="${joint_limits_parameters_file}"
@@ -26,5 +22,5 @@
       physical_parameters_file="${physical_parameters_file}"
       visual_parameters_file="${visual_parameters_file}"
-      use_fake_hardware="${use_fake_hardware}"
+      use_fake_hardware="false"
       use_tool_communication="true"
       generate_ros2_control_tag="true"
@@ -34,6 +30,6 @@
     <xacro:hande_gripper
       name="hande_gripper"
-      prefix="${gripper_prefix}"
-      parent="${ur_prefix}tool0"
+      prefix=""
+      parent="tool0"
       grip_pos_min="0"
       grip_pos_max="0.025"

File: ur10e_hande_moveit_config/config/ur10e_hande_robot.ros2_control.xacro (robot description, xacro)
@@ -1,57 +1,72 @@
 <?xml version="1.0"?>
-<robot xmlns:xacro="http://www.ros.org/wiki/xacro">
-    <xacro:macro name="ur10e_hande_robot_ros2_control" params="name initial_positions_file">
+<robot xmlns:xacro="http://ros.org/wiki/xacro">
+    <xacro:macro name="ur10e_hande_robot_ros2_control" params="name initial_positions_file use_fake_hardware">
         <xacro:property name="initial_positions" value="${load_yaml(initial_positions_file)['initial_positions']}"/>
         <ros2_control name="${name}" type="system">
             <hardware>
-                <!-- By default, set up controllers for simulation. This won't work on real hardware -->
-                <plugin>mock_components/GenericSystem</plugin>
+                <xacro:if value="${use_fake_hardware}">
+                    <plugin>mock_components/GenericSystem</plugin>
+                </xacro:if>
+                <xacro:unless value="${use_fake_hardware}">
+                    <!-- 실제 하드웨어에서는 UR 드라이버가 UR 조인트를 관리 -->
+                    <!-- 그리퍼는 별도 드라이버에서 관리 -->
+                    <plugin>mock_components/GenericSystem</plugin>
+                </xacro:unless>
             </hardware>
-            <joint name="ur_shoulder_pan_joint">
+            <!-- UR 조인트들 -->
+            <joint name="shoulder_pan_joint">
                 <command_interface name="position"/>
                 <state_interface name="position">
-                  <param name="initial_value">${initial_positions['ur_shoulder_pan_joint']}</param>
+                  <param name="initial_value">${initial_positions['shoulder_pan_joint']}</param>
                 </state_interface>
                 <state_interface name="velocity"/>
             </joint>
-            <joint name="ur_shoulder_lift_joint">
+            <joint name="shoulder_lift_joint">
                 <command_interface name="position"/>
                 <state_interface name="position">
-                  <param name="initial_value">${initial_positions['ur_shoulder_lift_joint']}</param>
+                  <param name="initial_value">${initial_positions['shoulder_lift_joint']}</param>
                 </state_interface>
                 <state_interface name="velocity"/>
             </joint>
-            <joint name="ur_elbow_joint">
+            <joint name="elbow_joint">
                 <command_interface name="position"/>
                 <state_interface name="position">
-                  <param name="initial_value">${initial_positions['ur_elbow_joint']}</param>
+                  <param name="initial_value">${initial_positions['elbow_joint']}</param>
                 </state_interface>
                 <state_interface name="velocity"/>
             </joint>
-            <joint name="ur_wrist_1_joint">
+            <joint name="wrist_1_joint">
                 <command_interface name="position"/>
                 <state_interface name="position">
-                  <param name="initial_value">${initial_positions['ur_wrist_1_joint']}</param>
+                  <param name="initial_value">${initial_positions['wrist_1_joint']}</param>
                 </state_interface>
                 <state_interface name="velocity"/>
             </joint>
-            <joint name="ur_wrist_2_joint">
+            <joint name="wrist_2_joint">
                 <command_interface name="position"/>
                 <state_interface name="position">
-                  <param name="initial_value">${initial_positions['ur_wrist_2_joint']}</param>
+                  <param name="initial_value">${initial_positions['wrist_2_joint']}</param>
                 </state_interface>
                 <state_interface name="velocity"/>
             </joint>
-            <joint name="ur_wrist_3_joint">
+            <joint name="wrist_3_joint">
                 <command_interface name="position"/>
                 <state_interface name="position">
-                  <param name="initial_value">${initial_positions['ur_wrist_3_joint']}</param>
+                  <param name="initial_value">${initial_positions['wrist_3_joint']}</param>
                 </state_interface>
                 <state_interface name="velocity"/>
             </joint>
-            <joint name="gr_hande_left_finger_joint">
+            <!-- Hande 그리퍼 조인트 (2F-140 드라이버와 호환) -->
+            <joint name="hande_left_finger_joint">
                 <command_interface name="position"/>
                 <state_interface name="position">
-                  <param name="initial_value">${initial_positions['gr_hande_left_finger_joint']}</param>
+                  <param name="initial_value">${initial_positions['hande_left_finger_joint']}</param>
+                </state_interface>
+                <state_interface name="velocity"/>
+            </joint>
+            <joint name="hande_right_finger_joint">
+                <command_interface name="position"/>
+                <state_interface name="position">
+                  <param name="initial_value">${initial_positions['hande_left_finger_joint']}</param>
                 </state_interface>
                 <state_interface name="velocity"/>
